File: electoronics/Octave_Input_PCB/Octave_Input_PCB.kicad_pcb (KiCad board)
At the start: 2 copper layers, 95.2 x 95.2 mm, 28 parts, among them SW1 SW_Hot_Swap_Socket, SW10 SW_Hot_Swap_Socket, SW11 SW_Hot_Swap_Socket, SW12 SW_Hot_Swap_Socket, SW13 SW_Hot_Swap_Socket, SW14 SW_Hot_Swap_Socket, SW2 SW_Hot_Swap_Socket, SW3 SW_Hot_Swap_Socket, SW4 SW_Hot_Swap_Socket, SW5 SW_Hot_Swap_Socket, SW6 SW_Hot_Swap_Socket, SW7 SW_Hot_Swap_Socket, SW8 SW_Hot_Swap_Socket, SW9 SW_Hot_Swap_Socket

Commit message: Update schematic and PCB
Routing:
- net row0: track 0.00 -> 69.6 mm, vias 0 -> 6
- net row2: track 0.00 -> 66.5 mm, vias 0 -> 6
- net row1: track 0.00 -> 66.4 mm, vias 0 -> 6
- net row3: track 0.00 -> 59.6 mm
- net col3: track 0.00 -> 57.2 mm
- net col0: track 0.00 -> 57.2 mm
- net col2: track 0.00 -> 38.1 mm
- net col1: track 0.00 -> 38.1 mm

Commit message: Update schematic
Parts:
- added U1: Adafruit_QT_Py_RP2040, Octave_Library:Adafruit_QT_Py_RP2040, F.Cu at (85.7, 114.3)
- D1, D10, D11, D12, D13, D14, D2, D3, D4, D5, D6, D7, D8, D9, SW1, SW10, SW11, SW12, SW13, SW14, SW2, SW3, SW4, SW5, SW6, SW7, SW8, SW9: moved to F.Cu
- moved D12 63.4 mm to (54.0, 95.2)
- moved D14 63.4 mm to (54.0, 114.3)
- moved D4 63.4 mm to (54.0, 57.1)
- moved D8 63.4 mm to (54.0, 76.2)
- moved SW1 57.1 mm to (114.3, 57.1), turned to 0 degrees
- moved SW12 57.1 mm to (57.1, 95.2), turned to 0 degrees
- moved SW13 57.1 mm to (114.3, 114.3), turned to 0 degrees
- moved SW14 57.1 mm to (57.1, 114.3), turned to 0 degrees
- moved SW4 57.1 mm to (57.1, 57.1), turned to 0 degrees
- moved SW5 57.1 mm to (114.3, 76.2), turned to 0 degrees
- moved SW8 57.1 mm to (57.1, 76.2), turned to 0 degrees
- moved SW9 57.1 mm to (114.3, 95.2), turned to 0 degrees
- moved D1 50.9 mm to (111.2, 57.1)
- moved D13 50.9 mm to (111.2, 114.3)
- moved D5 50.9 mm to (111.2, 76.2)
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Routing:
- net col0: track 57.2 -> 92.2 mm
- net col1: track 38.1 -> 72.1 mm
- net col2: track 38.1 -> 54.1 mm
- net col3: track 57.2 -> 70.7 mm

Commit message: Update schematic
Parts:
- added C1: 0.01u, Octave_Library:C_0805_2012Metric_Pad1.18x1.45mm_HandSolder, F.Cu at (104.8, 113.0)
- added C2: 0.01u, Octave_Library:C_0805_2012Metric_Pad1.18x1.45mm_HandSolder, F.Cu at (104.8, 118.1)
- added R1: 10K, Octave_Library:R_0805_2012Metric_Pad1.20x1.40mm_HandSolder, F.Cu at (97.2, 113.0)
- added R2: 10K, Octave_Library:R_0805_2012Metric_Pad1.20x1.40mm_HandSolder, F.Cu at (99.7, 113.0)
- added R3: 10K, Octave_Library:R_0805_2012Metric_Pad1.20x1.40mm_HandSolder, F.Cu at (97.2, 118.1)
- added R4: 10K, Octave_Library:R_0805_2012Metric_Pad1.20x1.40mm_HandSolder, F.Cu at (99.7, 118.1)
- SW13: value SW_Hot_Swap_Socket -> Bourns_PEC12R-4xxxF-Sxxx; footprint Octave_Library:Hot_Swap_Socket_CPG151101S11 -> Octave_Library:Incremental_Encoder_PEC12R-4xxxF-Sxxxx; moved to B.Cu
- moved D13 14.5 mm to (98.4, 107.3), turned to 0 degrees
- turned SW13 to 180 degrees
Connections:
- SW13 pad 1: Net-(D13-Pad2) -> col0
- SW13 pad 2: col0 -> Net-(D13-Pad2)
- U1 pad 10: row1 -> unconnected-(U1-Pad10)
- U1 pad 11: row0 -> SignalB
- U1 pad 12: unconnected-(U1-Pad12) -> +3V3
- U1 pad 13: unconnected-(U1-Pad13) -> C
- U1 pad 3: col3 -> col0
- U1 pad 4: unconnected-(U1-Pad4) -> row2
- U1 pad 5: unconnected-(U1-Pad5) -> col3
- U1 pad 6: unconnected-(U1-Pad6) -> row1
- U1 pad 7: unconnected-(U1-Pad7) -> row0
- U1 pad 8: col0 -> row3
- U1 pad 9: row2 -> SignalA
Routing:
- net row0: track 69.6 -> 164.7 mm
- net row1: track 66.4 -> 140.1 mm
- net C: track 0.00 -> 49.9 mm
- net B: track 0.00 -> 22.4 mm
- net A: track 0.00 -> 20.4 mm
- net row2: track 66.5 -> 86.3 mm
- net +3V3: track 0.00 -> 13.4 mm
- net Net-(D13-Pad2): track 5.26 -> 12.3 mm
- net SignalB: track 0.00 -> 6.46 mm
- net SignalA: track 0.00 -> 6.46 mm
- net col0: track 92.2 -> 98.2 mm
- net col3: track 70.7 -> 72.7 mm
- net row3: track 59.6 -> 60.9 mm
