File: electronics/Octave_Input_PCB/Octave_Input_PCB.kicad_pcb (KiCad board)
At the start: 2 copper layers, 87.8 x 95.8 mm, 66 parts, among them J1 HRO_TYPE-C-31-M-12, SW1 SW_Hot_Swap_Socket, SW10 SW_Hot_Swap_Socket, SW11 SW_Hot_Swap_Socket, SW12 SW_Hot_Swap_Socket, SW13 SW_Hot_Swap_Socket, SW14 Alps_Alpine_RKJXV1224, SW15 Bourns_PEC12R-4xxxF-Sxxx, SW2 SW_Hot_Swap_Socket, SW21 Alps_Alpine_SKRP, SW22 Alps_Alpine_SKRP, SW3 SW_Hot_Swap_Socket, SW4 SW_Hot_Swap_Socket, SW5 SW_Hot_Swap_Socket, SW6 SW_Hot_Swap_Socket, SW7 SW_Hot_Swap_Socket, SW8 SW_Hot_Swap_Socket, SW9 SW_Hot_Swap_Socket, U1 AP2112K-3.3, U2 Raspberry_Pi_RP2040, U3 W25Q64JVSS, Y1 12MHz

Commit message: [WIP] Update schematic and PCB
Parts:
- moved R12 11.3 mm to (59.6, 117.2), turned to 180 degrees
- moved C21 8.07 mm to (56.6, 119.9)
- moved R14 7.99 mm to (59.6, 118.3), turned to 0 degrees
- moved C22 7.36 mm to (57.6, 119.9)
Connections:
- U2 pad 34: col0 -> row3
- U2 pad 36: row3 -> col0
- U2 pad 38: stickA -> stickB
- U2 pad 39: stickB -> stickA
Routing:
- net row3: track 0.00 -> 66.4 mm, vias 0 -> 4
- net row0: track 62.2 -> 121.2 mm, vias 6 -> 8
- net col0: track 57.2 -> 91.1 mm, vias 0 -> 2
- net stickB: track 0.00 -> 27.5 mm, vias 0 -> 1
- net stickA: track 0.00 -> 19.9 mm, vias 0 -> 1
- net col1: track 97.5 -> 109.5 mm
- net B: track 0.00 -> 3.17 mm
- net A: track 0.00 -> 3.17 mm
- net +3V3: track 136.6 -> 135.4 mm
- net row1: track 99.2 -> 99.8 mm

Commit message: Update schematic and PCB
Parts:
- moved D15 19.0 mm to (54.6, 114.3), turned to 90 degrees
- moved R11 18.2 mm to (75.3, 102.6), turned to 0 degrees
- moved R13 16.2 mm to (75.3, 103.6), turned to 0 degrees
- moved R12 2.06 mm to (61.1, 118.7)
- moved R14 1.99 mm to (61.1, 119.7)
- moved C22 1.55 mm to (59.2, 119.7), turned to 180 degrees
- moved C21 1.55 mm to (55.1, 119.7), turned to 0 degrees
Connections:
- U2 pad 4: rotaryA -> rotaryB
- U2 pad 5: rotaryB -> rotaryA
Routing:
- net rotaryB: track 0.00 -> 33.5 mm
- net rotaryA: track 0.00 -> 32.5 mm
- net row3: track 66.4 -> 86.2 mm, vias 4 -> 6
- net +3V3: track 135.4 -> 146.3 mm, vias 6 -> 8
- net Net-(D15-Pad2): track 0.00 -> 5.90 mm
- net B: track 3.17 -> 8.51 mm
- net GND: track 26.3 -> 31.5 mm
- net col3: track 80.9 -> 79.3 mm
- added copper zone on F.Cu, net GND

Commit message: Complete schematic and PCB (rev.5.0.0)
Parts:
- added LED1: WS2812C-2020-V1, Octave_Library:WS2812C-2020, F.Cu at (76.2, 107.9)
- added REF**: M2, MountingHole:MountingHole_2.2mm_M2_ISO14580, F.Cu at (47.6, 47.6)
- added REF**: M2, MountingHole:MountingHole_2.2mm_M2_ISO14580, F.Cu at (123.8, 131.8)
- added REF**: M2, MountingHole:MountingHole_2.2mm_M2_ISO14580, F.Cu at (47.6, 123.8)
- added REF**: M2, MountingHole:MountingHole_2.2mm_M2_ISO14580, F.Cu at (123.8, 123.8)
- added REF**: M2, MountingHole:MountingHole_2.2mm_M2_ISO14580, F.Cu at (123.8, 47.6)
- added REF**: M2, MountingHole:MountingHole_2.2mm_M2_ISO14580, F.Cu at (47.6, 131.8)
Routing:
- net NEOPIX: track 0.00 -> 6.27 mm
- net NEOPIX_POWER: track 0.00 -> 5.17 mm
- net GND: track 31.5 -> 32.4 mm, vias 24 -> 54
Other:
- board text added: "Octave Input PCB rev.5.0.0"
- board text removed: "Octave Input PCB rev.5.a"

Commit message: Fix C13 and C14 value, improve Y1 pattern
Parts:
- removed REF** (x6): M2, MountingHole:MountingHole_2.2mm_M2_ISO14580
- C13, C14: value 1uF -> 0.1uF
Other:
- board text added: "Octave Input PCB rev.5.0.1"
- board text removed: "Octave Input PCB rev.5.0.0"
Changed lines of the file:
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@@
   (title_block
     (title "Octave - Input PCB")
-    (date "2022-05-29")
-    (rev "5.0.0")
+    (date "2022-05-30")
+    (rev "5.0.1")
     (comment 4 "https://github.com/takayoshiotake/octave-12-key-macropad")
   )
@@
     )
     (pad_to_mask_clearance 0)
+    (grid_origin 82.425 111.08)
     (pcbplotparams
       (layerselection 0x00010fc_ffffffff)
       (disableapertmacros false)
       (usegerberextensions false)
-      (usegerberattributes true)
-      (usegerberadvancedattributes true)
-      (creategerberjobfile true)
+      (usegerberattributes false)
+      (usegerberadvancedattributes false)
+      (creategerberjobfile false)
       (svguseinch false)
       (svgprecision 6)
@@
     )
   )
-  (footprint "MountingHole:MountingHole_2.2mm_M2_ISO14580" (layer "F.Cu")
-    (at 47.625 47.625)
-    (descr "Mounting Hole 2.2mm, no annular, M2, ISO14580")
-    (tags "mounting hole 2.2mm no annular m2 iso14580")
-    (attr exclude_from_pos_files exclude_from_bom)
-    (fp_text reference "REF**" (at 0 -2.9) (layer "F.SilkS") hide
-      (effects (font (size 1 1) (thickness 0.15)))
-    )
-    (fp_text value "M2" (at 0 2.9) (layer "F.Fab")
-      (effects (font (size 1 1) (thickness 0.15)))
-    )
-    (fp_text user "${REFERENCE}" (at 0 0) (layer "F.Fab") hide
-      (effects (font (size 1 1) (thickness 0.15)))
-    )
-    (fp_circle (center 0 0) (end 1.9 0) (layer "Cmts.User") (width 0.15) (fill none))
-    (fp_circle (center 0 0) (end 2.15 0) (layer "F.CrtYd") (width 0.05) (fill none))
-    (pad "" np_thru_hole circle (at 0 0) (size 2.2 2.2) (drill 2.2) (layers *.Cu *.Mask))
-  )
   (footprint "Octave_Library:RP2040_QFN-56" locked (layer "F.Cu")
     (at 85.725 104.775)
@@
       (effects (font (size 1 1) (thickness 0.15)))
     )
-    (fp_text value "1uF" (at 0 1.16) (layer "F.Fab") hide
+    (fp_text value "0.1uF" (at 0 1.16) (layer "F.Fab") hide
       (effects (font (size 1 1) (thickness 0.15)))
     )
@@
       (effects (font (size 1 1) (thickness 0.15)))
     )
-    (fp_text value "1uF" (at 0 1.16 90) (layer "F.Fab") hide
+    (fp_text value "0.1uF" (at 0 1.16 90) (layer "F.Fab") hide
       (effects (font (size 1 1) (thickness 0.15)))
     )
@@
     (pad "MP" thru_hole oval (at -4.32 -1.6325 180) (size 1 2.1) (drill oval 0.6 1.7) (layers *.Cu *.Mask))
   )
-  (footprint "MountingHole:MountingHole_2.2mm_M2_ISO14580" (layer "F.Cu")
-    (at 123.825 131.825)
-    (descr "Mounting Hole 2.2mm, no annular, M2, ISO14580")
-    (tags "mounting hole 2.2mm no annular m2 iso14580")
-    (attr exclude_from_pos_files exclude_from_bom)
-    (fp_text reference "REF**" (at 0 -2.9) (layer "F.SilkS") hide
-      (effects (font (size 1 1) (thickness 0.15)))
-    )
-    (fp_text value "M2" (at 0 2.9) (layer "F.Fab")
-      (effects (font (size 1 1) (thickness 0.15)))
-    )
-    (fp_text user "${REFERENCE}" (at 0 0) (layer "F.Fab") hide
-      (effects (font (size 1 1) (thickness 0.15)))
-    )
-    (fp_circle (center 0 0) (end 1.9 0) (layer "Cmts.User") (width 0.15) (fill none))
-    (fp_circle (center 0 0) (end 2.15 0) (layer "F.CrtYd") (width 0.05) (fill none))
-    (pad "" np_thru_hole circle (at 0 0) (size 2.2 2.2) (drill 2.2) (layers *.Cu *.Mask))
-  )
   (footprint "Capacitor_SMD:C_0402_1005Metric" (layer "F.Cu")
     (at 79.265 111.93 180)
@@
     )
   )
-  (footprint "MountingHole:MountingHole_2.2mm_M2_ISO14580" (layer "F.Cu")
-    (at 47.625 123.825)
-    (descr "Mounting Hole 2.2mm, no annular, M2, ISO14580")
-    (tags "mounting hole 2.2mm no annular m2 iso14580")
-    (attr exclude_from_pos_files exclude_from_bom)
-    (fp_text reference "REF**" (at 0 -2.9) (layer "F.SilkS") hide
-      (effects (font (size 1 1) (thickness 0.15)))
-    )
-    (fp_text value "M2" (at 0 2.9) (layer "F.Fab")
-      (effects (font (size 1 1) (thickness 0.15)))
-    )
-    (fp_text user "${REFERENCE}" (at 0 0) (layer "F.Fab") hide
-      (effects (font (size 1 1) (thickness 0.15)))
-    )
-    (fp_circle (center 0 0) (end 1.9 0) (layer "Cmts.User") (width 0.15) (fill none))
-    (fp_circle (center 0 0) (end 2.15 0) (layer "F.CrtYd") (width 0.05) (fill none))
-    (pad "" np_thru_hole circle (at 0 0) (size 2.2 2.2) (drill 2.2) (layers *.Cu *.Mask))
-  )
   (footprint "Resistor_SMD:R_0402_1005Metric" locked (layer "F.Cu")
     (at 88.135 110.43 90)
@@
     )
   )
-  (footprint "MountingHole:MountingHole_2.2mm_M2_ISO14580" (layer "F.Cu")
-    (at 123.825 123.825)
-    (descr "Mounting Hole 2.2mm, no annular, M2, ISO14580")
-    (tags "mounting hole 2.2mm no annular m2 iso14580")
-    (attr exclude_from_pos_files exclude_from_bom)
-    (fp_text reference "REF**" (at 0 -2.9) (layer "F.SilkS") hide
-      (effects (font (size 1 1) (thickness 0.15)))
-    )
-    (fp_text value "M2" (at 0 2.9) (layer "F.Fab")
-      (effects (font (size 1 1) (thickness 0.15)))
-    )
-    (fp_text user "${REFERENCE}" (at 0 0) (layer "F.Fab") hide
-      (effects (font (size 1 1) (thickness 0.15)))
-    )
-    (fp_circle (center 0 0) (end 1.9 0) (layer "Cmts.User") (width 0.15) (fill none))
-    (fp_circle (center 0 0) (end 2.15 0) (layer "F.CrtYd") (width 0.05) (fill none))
-    (pad "" np_thru_hole circle (at 0 0) (size 2.2 2.2) (drill 2.2) (layers *.Cu *.Mask))
-  )
   (footprint "Octave_Library:D_SOD-323F" (layer "F.Cu")
     (at 92.1258 76.2 90)
@@
     )
   )
-  (footprint "MountingHole:MountingHole_2.2mm_M2_ISO14580" (layer "F.Cu")
-    (at 123.825 47.625)
-    (descr "Mounting Hole 2.2mm, no annular, M2, ISO14580")
-    (tags "mounting hole 2.2mm no annular m2 iso14580")
-    (attr exclude_from_pos_files exclude_from_bom)
-    (fp_text reference "REF**" (at 0 -2.9) (layer "F.SilkS") hide
-      (effects (font (size 1 1) (thickness 0.15)))
-    )
-    (fp_text value "M2" (at 0 2.9) (layer "F.Fab")
-      (effects (font (size 1 1) (thickness 0.15)))
-    )
-    (fp_text user "${REFERENCE}" (at 0 0) (layer "F.Fab") hide
-      (effects (font (size 1 1) (thickness 0.15)))
-    )
-    (fp_circle (center 0 0) (end 1.9 0) (layer "Cmts.User") (width 0.15) (fill none))
-    (fp_circle (center 0 0) (end 2.15 0) (layer "F.CrtYd") (width 0.05) (fill none))
-    (pad "" np_thru_hole circle (at 0 0) (size 2.2 2.2) (drill 2.2) (layers *.Cu *.Mask))
-  )
   (footprint "Octave_Library:Hot_Swap_Socket_CPG151101S11" (layer "F.Cu")
     (at 114.3 95.25)
@@
     )
   )
-  (footprint "MountingHole:MountingHole_2.2mm_M2_ISO14580" (layer "F.Cu")
-    (at 47.625 131.825)
-    (descr "Mounting Hole 2.2mm, no annular, M2, ISO14580")
-    (tags "mounting hole 2.2mm no annular m2 iso14580")
-    (attr exclude_from_pos_files exclude_from_bom)
-    (fp_text reference "REF**" (at 0 -2.9) (layer "F.SilkS") hide
-      (effects (font (size 1 1) (thickness 0.15)))
-    )
-    (fp_text value "M2" (at 0 2.9) (layer "F.Fab")
-      (effects (font (size 1 1) (thickness 0.15)))
-    )
-    (fp_text user "${REFERENCE}" (at 0 0) (layer "F.Fab") hide
-      (effects (font (size 1 1) (thickness 0.15)))
-    )
-    (fp_circle (center 0 0) (end 1.9 0) (layer "Cmts.User") (width 0.15) (fill none))
-    (fp_circle (center 0 0) (end 2.15 0) (layer "F.CrtYd") (width 0.05) (fill none))
-    (pad "" np_thru_hole circle (at 0 0) (size 2.2 2.2) (drill 2.2) (layers *.Cu *.Mask))
-  )
   (footprint "Capacitor_SMD:C_0402_1005Metric" locked (layer "F.Cu")
     (at 86.135 110.41 -90)
@@
     (effects (font (size 1 1) (thickness 0.15)) (justify right))
   )
-  (gr_text "Octave Input PCB rev.5.0.0" (at 50.725 135.725) (layer "F.SilkS")
+  (gr_text "Octave Input PCB rev.5.0.1" (at 50.725 135.725) (layer "F.SilkS")
     (effects (font (size 1 1) (thickness 0.15)) (justify left))
   )
@@
   (segment (start 76.2 103.555) (end 76.42 103.775) (width 0.2) (layer "F.Cu") (net 75))
   (segment (start 76.42 103.775) (end 82.2875 103.775) (width 0.2) (layer "F.Cu") (net 75))
+  (zone (net 0) (net_name "") (layer "F.Cu") (hatch edge 0.508)
+    (connect_pads yes (clearance 0))
+    (min_thickness 0.4)
+    (keepout (tracks allowed) (vias allowed) (pads allowed ) (copperpour not_allowed) (footprints allowed))
+    (fill (thermal_gap 0.508) (thermal_bridge_width 0.508))
+    (polygon
+      (pts
+        (xy 85.625 113.28)
+        (xy 79.265 113.28)
+        (xy 79.265 108.78)
+        (xy 85.625 108.78)
+      )
+    )
+  )
   (zone locked (net 22) (net_name "+3V3") (layer "F.Cu") (hatch full 0.508)
     (priority 1)

Commit message: Add pull-up for QSPI_SS_N
Parts:
- added R6: 10K, Resistor_SMD:R_0402_1005Metric, F.Cu at (63.3, 110.1)
- renumbered R6 to R7, R7 to R8
Routing:
- net +3V3: track 146.3 -> 156.1 mm
- net QSPI_SS_N: track 23.9 -> 24.9 mm
- net GND: vias 54 -> 57
Changed lines of the file:
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@@
   (net 68 "Net-(C15-Pad1)")
   (net 69 "Net-(C16-Pad1)")
-  (net 70 "Net-(R7-Pad1)")
+  (net 70 "Net-(R8-Pad1)")
   (net 71 "~{USB_BOOT}")
   (net 72 "~{RESET}")
@@
     (property "Sheetname" "")
     (attr smd)
-    (fp_text reference "R7" (at 0 -1.17 90) (layer "F.SilkS") hide
+    (fp_text reference "R8" (at 0 -1.17 90) (layer "F.SilkS") hide
       (effects (font (size 1 1) (thickness 0.15)))
     )
@@
     (fp_line (start 0.525 -0.27) (end 0.525 0.27) (layer "F.Fab") (width 0.1))
     (pad "1" smd roundrect (at -0.51 0 270) (size 0.54 0.64) (layers "F.Cu" "F.Paste" "F.Mask") (roundrect_rratio 0.25)
-      (net 70 "Net-(R7-Pad1)") (pintype "passive"))
+      (net 70 "Net-(R8-Pad1)") (pintype "passive"))
     (pad "2" smd roundrect (at 0.51 0 270) (size 0.54 0.64) (layers "F.Cu" "F.Paste" "F.Mask") (roundrect_rratio 0.25)
       (net 69 "Net-(C16-Pad1)") (pintype "passive"))
@@
       (net 68 "Net-(C15-Pad1)") (pinfunction "XIN") (pintype "input"))
     (pad "21" smd roundrect locked (at -0.2 3.4375 90) (size 0.875 0.2) (layers "F.Cu" "F.Paste" "F.Mask") (roundrect_rratio 0.25)
-      (net 70 "Net-(R7-Pad1)") (pinfunction "XOUT") (pintype "passive"))
+      (net 70 "Net-(R8-Pad1)") (pinfunction "XOUT") (pintype "passive"))
     (pad "22" smd roundrect locked (at 0.2 3.4375 90) (size 0.875 0.2) (layers "F.Cu" "F.Paste" "F.Mask") (roundrect_rratio 0.25)
       (net 22 "+3V3") (pinfunction "IOVDD") (pintype "power_in"))
@@
     )
   )
+  (footprint "Resistor_SMD:R_0402_1005Metric" (layer "F.Cu")
+    (at 63.26 110.095)
+    (descr "Resistor SMD 0402 (1005 Metric), square (rectangular) end terminal, IPC_7351 nominal, (Body size source: IPC-SM-782 page 72, https://www.pcb-3d.com/wordpress/wp-content/uploads/ipc-sm-782a_amendment_1_and_2.pdf), generated with kicad-footprint-generator")
+    (tags "resistor")
+    (property "Sheetfile" "Octave_Input_PCB.kicad_sch")
+    (property "Sheetname" "")
+    (attr smd)
+    (fp_text reference "R6" (at 0 -1.17) (layer "F.SilkS") hide
+      (effects (font (size 1 1) (thickness 0.15)))
+    )
+    (fp_text value "10K" (at 0 1.17) (layer "F.Fab") hide
+      (effects (font (size 1 1) (thickness 0.15)))
+    )
+    (fp_text user "${REFERENCE}" (at 0 0) (layer "F.Fab")
+      (effects (font (size 0.26 0.26) (thickness 0.04)))
+    )
+    (fp_line (start -0.153641 -0.38) (end 0.153641 -0.38) (layer "F.SilkS") (width 0.12))
+    (fp_line (start -0.153641 0.38) (end 0.153641 0.38) (layer "F.SilkS") (width 0.12))
+    (fp_line (start -0.93 -0.47) (end 0.93 -0.47) (layer "F.CrtYd") (width 0.05))
+    (fp_line (start 0.93 0.47) (end -0.93 0.47) (layer "F.CrtYd") (width 0.05))
+    (fp_line (start 0.93 -0.47) (end 0.93 0.47) (layer "F.CrtYd") (width 0.05))
+    (fp_line (start -0.93 0.47) (end -0.93 -0.47) (layer "F.CrtYd") (width 0.05))
+    (fp_line (start 0.525 0.27) (end -0.525 0.27) (layer "F.Fab") (width 0.1))
+    (fp_line (start 0.525 -0.27) (end 0.525 0.27) (layer "F.Fab") (width 0.1))
+    (fp_line (start -0.525 0.27) (end -0.525 -0.27) (layer "F.Fab") (width 0.1))
+    (fp_line (start -0.525 -0.27) (end 0.525 -0.27) (layer "F.Fab") (width 0.1))
+    (pad "1" smd roundrect (at -0.51 0) (size 0.54 0.64) (layers "F.Cu" "F.Paste" "F.Mask") (roundrect_rratio 0.25)
+      (net 22 "+3V3") (pintype "passive"))
+    (pad "2" smd roundrect (at 0.51 0) (size 0.54 0.64) (layers "F.Cu" "F.Paste" "F.Mask") (roundrect_rratio 0.25)
+      (net 65 "QSPI_SS_N") (pintype "passive"))
+    (model "${KICAD6_3DMODEL_DIR}/Resistor_SMD.3dshapes/R_0402_1005Metric.wrl"
+      (offset (xyz 0 0 0))
+      (scale (xyz 1 1 1))
+      (rotate (xyz 0 0 0))
+    )
+  )
   (footprint "Octave_Library:D_SOD-323F" locked (layer "F.Cu")
     (at 54.65 114.3 90)
@@
     )
   )
-  (footprint "Resistor_SMD:R_0402_1005Metric" (layer "F.Cu")
+  (footprint "Resistor_SMD:R_0402_1005Metric" locked (layer "F.Cu")
     (at 65.28 110.095)
     (descr "Resistor SMD 0402 (1005 Metric), square (rectangular) end terminal, IPC_7351 nominal, (Body size source: IPC-SM-782 page 72, https://www.pcb-3d.com/wordpress/wp-content/uploads/ipc-sm-782a_amendment_1_and_2.pdf), generated with kicad-footprint-generator")
@@
     (property "Sheetname" "")
     (attr smd)
-    (fp_text reference "R6" (at 0 -1.17) (layer "F.SilkS") hide
+    (fp_text reference "R7" (at 0 -1.17) (layer "F.SilkS") hide
       (effects (font (size 1 1) (thickness 0.15)))
     )
@@
     (fp_line (start -0.525 0.27) (end -0.525 -0.27) (layer "F.Fab") (width 0.1))
     (fp_line (start 0.525 -0.27) (end 0.525 0.27) (layer "F.Fab") (width 0.1))
-    (pad "1" smd roundrect (at -0.51 0) (size 0.54 0.64) (layers "F.Cu" "F.Paste" "F.Mask") (roundrect_rratio 0.25)
+    (pad "1" smd roundrect locked (at -0.51 0) (size 0.54 0.64) (layers "F.Cu" "F.Paste" "F.Mask") (roundrect_rratio 0.25)
       (net 65 "QSPI_SS_N") (pintype "passive"))
-    (pad "2" smd roundrect (at 0.51 0) (size 0.54 0.64) (layers "F.Cu" "F.Paste" "F.Mask") (roundrect_rratio 0.25)
+    (pad "2" smd roundrect locked (at 0.51 0) (size 0.54 0.64) (layers "F.Cu" "F.Paste" "F.Mask") (roundrect_rratio 0.25)
       (net 71 "~{USB_BOOT}") (pintype "passive"))
     (model "${KICAD6_3DMODEL_DIR}/Resistor_SMD.3dshapes/R_0402_1005Metric.wrl"
@@
   (segment (start 66.445 98.6) (end 82.725 98.6) (width 0.2) (layer "F.Cu") (net 22))
   (segment (start 83.725 103.175) (end 84.125 102.775) (width 0.2) (layer "F.Cu") (net 22))
+  (segment (start 62.75 110.095) (end 62.75 103.195) (width 0.4) (layer "F.Cu") (net 22))
   (segment (start 90.5 105.975) (end 90.3 105.775) (width 0.2) (layer "F.Cu") (net 22))
   (segment (start 88.325 105.775) (end 88.325 103.175) (width 0.2) (layer "F.Cu") (net 22))
@@
   (segment (start 85.225 106.775) (end 85.725 107.275) (width 0.2) (layer "F.Cu") (net 22))
   (segment (start 89.325 100.6) (end 88.125 100.6) (width 0.2) (layer "F.Cu") (net 22))
+  (segment (start 62.75 103.195) (end 64.77 101.175) (width 0.4) (layer "F.Cu") (net 22))
   (segment (start 88.025 102.275) (end 88.025 102.875) (width 0.2) (layer "F.Cu") (net 22))
   (segment (start 85.925 107.475) (end 85.725 107.275) (width 0.2) (layer "F.Cu") (net 22))
@@
   (segment (start 78.83 101.975) (end 79.61 101.975) (width 0.2) (layer "F.Cu") (net 26))
   (segment (start 84.925 97.26) (end 84.925 96.48) (width 0.2) (layer "F.Cu") (net 26))
+  (via (at 63.65 107.075) (size 0.6) (drill 0.3) (layers "F.Cu" "B.Cu") (remove_unused_layers) (keep_end_layers) (net 26))
   (via (at 119.0625 90.4875) (size 0.6) (drill 0.3) (layers "F.Cu" "B.Cu") (remove_unused_layers) (keep_end_layers) (net 26))
   (via (at 74.435 108.475) (size 0.6) (drill 0.3) (layers "F.Cu" "B.Cu") (remove_unused_layers) (keep_end_layers) (net 26))
@@
   (via (at 100.0125 52.3875) (size 0.6) (drill 0.3) (layers "F.Cu" "B.Cu") (remove_unused_layers) (keep_end_layers) (net 26))
   (via (at 85.925 96.48) (size 0.6) (drill 0.3) (layers "F.Cu" "B.Cu") (remove_unused_layers) (keep_end_layers) (net 26))
+  (via (at 66.04 103.555) (size 0.6) (drill 0.3) (layers "F.Cu" "B.Cu") (remove_unused_layers) (keep_end_layers) (net 26))
   (via (at 109.5375 119.0625) (size 0.6) (drill 0.3) (layers "F.Cu" "B.Cu") (remove_unused_layers) (keep_end_layers) (net 26))
+  (via (at 71.625 100.48) (size 0.6) (drill 0.3) (layers "F.Cu" "B.Cu") (remove_unused_layers) (keep_end_layers) (net 26))
   (via (at 86.135 111.669999) (size 0.6) (drill 0.3) (layers "F.Cu" "B.Cu") (remove_unused_layers) (keep_end_layers) (net 26))
   (via (at 92.619999 100.975) (size 0.6) (drill 0.3) (layers "F.Cu" "B.Cu") (remove_unused_layers) (keep_end_layers) (net 26))
@@
   (segment (start 68.345 106.475) (end 73.82 101) (width 0.2) (layer "F.Cu") (net 65))
   (segment (start 73.82 101) (end 83.125 101) (width 0.2) (layer "F.Cu") (net 65))
+  (segment (start 63.77 110.095) (end 64.77 110.095) (width 0.2) (layer "F.Cu") (net 65))
   (segment (start 64.77 107.11) (end 65.405 106.475) (width 0.2) (layer "F.Cu") (net 65))
   (segment (start 83.645 110.23) (end 85.125 108.75) (width 0.2) (layer "F.Cu") (net 68))

Commit message: Change C1 and C2 value
Parts:
- C1, C2: value 1uF -> 10uF
Other:
- board text added: "Octave Input PCB rev.5.0.2"
- board text removed: "Octave Input PCB rev.5.0.1"
Changed lines of the file:
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@@
     (title "Octave - Input PCB")
     (date "2022-05-30")
-    (rev "5.0.1")
+    (rev "5.0.2")
     (comment 4 "https://github.com/takayoshiotake/octave-12-key-macropad")
   )
@@
       (effects (font (size 1 1) (thickness 0.15)))
     )
-    (fp_text value "1uF" (at 0 1.16) (layer "F.Fab") hide
+    (fp_text value "10uF" (at 0 1.16) (layer "F.Fab") hide
       (effects (font (size 1 1) (thickness 0.15)))
     )
@@
       (effects (font (size 1 1) (thickness 0.15)))
     )
-    (fp_text value "1uF" (at 0 1.16) (layer "F.Fab") hide
+    (fp_text value "10uF" (at 0 1.16) (layer "F.Fab") hide
       (effects (font (size 1 1) (thickness 0.15)))
     )
@@
     (effects (font (size 1 1) (thickness 0.15)) (justify right))
   )
-  (gr_text "Octave Input PCB rev.5.0.1" (at 50.725 135.725) (layer "F.SilkS")
+  (gr_text "Octave Input PCB rev.5.0.2" (at 50.725 135.725) (layer "F.SilkS")
     (effects (font (size 1 1) (thickness 0.15)) (justify left))
   )

Commit message: Rename footprint of tactile switch
Parts:
- SW21, SW22: footprint Octave_Library:Tactile_Switch_SKRP_ Series -> Octave_Library:Tactile_Switch_SKRP_Series
Changed lines of the file:
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@@
     )
   )
-  (footprint "Octave_Library:Tactile_Switch_SKRP_ Series" locked (layer "F.Cu")
+  (footprint "Octave_Library:Tactile_Switch_SKRP_Series" locked (layer "F.Cu")
     (at 100.0125 109.5375 90)
     (property "Sheetfile" "Octave_Input_PCB.kicad_sch")
@@
     (fp_line (start -0.4 -1.1) (end 0.4 -1.1) (layer "F.Fab") (width 0.1))
     (fp_rect (start -2.1 -1.6) (end 2.1 1.6) (layer "F.Fab") (width 0.1) (fill none))
+    (fp_arc (start 0.4 -1.1) (mid 1.5 0) (end 0.4 1.1) (layer "F.Fab") (width 0.1))
     (fp_arc (start -0.4 1.1) (mid -1.5 0) (end -0.4 -1.1) (layer "F.Fab") (width 0.1))
-    (fp_arc (start 0.4 -1.1) (mid 1.5 0) (end 0.4 1.1) (layer "F.Fab") (width 0.1))
     (pad "1" smd rect locked (at -2.075 -1.075 90) (size 1.05 0.65) (layers "F.Cu" "F.Paste" "F.Mask")
       (net 26 "GND") (pinfunction "1") (pintype "passive"))
@@
     )
   )
-  (footprint "Octave_Library:Tactile_Switch_SKRP_ Series" locked (layer "F.Cu")
+  (footprint "Octave_Library:Tactile_Switch_SKRP_Series" locked (layer "F.Cu")
     (at 71.4375 109.5375 90)
     (property "Sheetfile" "Octave_Input_PCB.kicad_sch")
@@
     )
     (fp_rect (start -2.8 -1.8) (end 2.8 1.8) (layer "F.CrtYd") (width 0.05) (fill none))
+    (fp_line (start -0.4 1.1) (end 0.4 1.1) (layer "F.Fab") (width 0.1))
     (fp_line (start -0.4 -1.1) (end 0.4 -1.1) (layer "F.Fab") (width 0.1))
-    (fp_line (start -0.4 1.1) (end 0.4 1.1) (layer "F.Fab") (width 0.1))
     (fp_rect (start -2.1 -1.6) (end 2.1 1.6) (layer "F.Fab") (width 0.1) (fill none))
     (fp_arc (start 0.4 -1.1) (mid 1.5 0) (end 0.4 1.1) (layer "F.Fab") (width 0.1))
