File: electronics/Octave_Input_PCB/Octave_Input_PCB.kicad_pcb (KiCad board)
At the start: 2 copper layers, 87.8 x 95.8 mm, 68 parts, among them J1 HRO_TYPE-C-31-M-12, SW1 SW_Hot_Swap_Socket, SW10 SW_Hot_Swap_Socket, SW11 SW_Hot_Swap_Socket, SW12 SW_Hot_Swap_Socket, SW13 SW_Hot_Swap_Socket, SW14 Alps_Alpine_RKJXV1224, SW15 Bourns_PEC12R-4xxxF-Sxxx, SW2 SW_Hot_Swap_Socket, SW21 Alps_Alpine_SKRP, SW22 Alps_Alpine_SKRP, SW3 SW_Hot_Swap_Socket, SW4 SW_Hot_Swap_Socket, SW5 SW_Hot_Swap_Socket, SW6 SW_Hot_Swap_Socket, SW7 SW_Hot_Swap_Socket, SW8 SW_Hot_Swap_Socket, SW9 SW_Hot_Swap_Socket, U1 AP2112K-3.3, U2 Raspberry_Pi_RP2040, U3 W25Q64JVSS, Y1 12MHz

Commit message: Fix
Parts:
- added REF**: M2, MountingHole:MountingHole_2.2mm_M2_ISO14580, F.Cu at (47.6, 131.8)
- added REF**: M2, MountingHole:MountingHole_2.2mm_M2_ISO14580, F.Cu at (47.6, 47.6)
- added REF**: M2, MountingHole:MountingHole_2.2mm_M2_ISO14580, F.Cu at (123.8, 47.6)
- added REF**: M2, MountingHole:MountingHole_2.2mm_M2_ISO14580, F.Cu at (47.6, 123.8)
- added REF**: M2, MountingHole:MountingHole_2.2mm_M2_ISO14580, F.Cu at (123.8, 131.8)
- added REF**: M2, MountingHole:MountingHole_2.2mm_M2_ISO14580, F.Cu at (123.8, 123.8)
Changed lines of the file:
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@@
     )
     (pad_to_mask_clearance 0)
-    (grid_origin 82.425 111.08)
     (pcbplotparams
       (layerselection 0x00010fc_ffffffff)
@@
     )
   )
+  (footprint "MountingHole:MountingHole_2.2mm_M2_ISO14580" (layer "F.Cu")
+    (at 47.625 131.825)
+    (descr "Mounting Hole 2.2mm, no annular, M2, ISO14580")
+    (tags "mounting hole 2.2mm no annular m2 iso14580")
+    (attr exclude_from_pos_files exclude_from_bom)
+    (fp_text reference "REF**" (at 0 -2.9) (layer "F.SilkS") hide
+      (effects (font (size 1 1) (thickness 0.15)))
+    )
+    (fp_text value "M2" (at 0 2.9) (layer "F.Fab")
+      (effects (font (size 1 1) (thickness 0.15)))
+    )
+    (fp_text user "${REFERENCE}" (at 0 0) (layer "F.Fab") hide
+      (effects (font (size 1 1) (thickness 0.15)))
+    )
+    (fp_circle (center 0 0) (end 1.9 0) (layer "Cmts.User") (width 0.15) (fill none))
+    (fp_circle (center 0 0) (end 2.15 0) (layer "F.CrtYd") (width 0.05) (fill none))
+    (pad "" np_thru_hole circle (at 0 0) (size 2.2 2.2) (drill 2.2) (layers *.Cu *.Mask))
+  )
   (footprint "Capacitor_SMD:C_0402_1005Metric" (layer "F.Cu")
     (at 84.925 97.74 90)
@@
     )
   )
+  (footprint "MountingHole:MountingHole_2.2mm_M2_ISO14580" (layer "F.Cu")
+    (at 47.625 47.625)
+    (descr "Mounting Hole 2.2mm, no annular, M2, ISO14580")
+    (tags "mounting hole 2.2mm no annular m2 iso14580")
+    (attr exclude_from_pos_files exclude_from_bom)
+    (fp_text reference "REF**" (at 0 -2.9) (layer "F.SilkS") hide
+      (effects (font (size 1 1) (thickness 0.15)))
+    )
+    (fp_text value "M2" (at 0 2.9) (layer "F.Fab")
+      (effects (font (size 1 1) (thickness 0.15)))
+    )
+    (fp_text user "${REFERENCE}" (at 0 0) (layer "F.Fab") hide
+      (effects (font (size 1 1) (thickness 0.15)))
+    )
+    (fp_circle (center 0 0) (end 1.9 0) (layer "Cmts.User") (width 0.15) (fill none))
+    (fp_circle (center 0 0) (end 2.15 0) (layer "F.CrtYd") (width 0.05) (fill none))
+    (pad "" np_thru_hole circle (at 0 0) (size 2.2 2.2) (drill 2.2) (layers *.Cu *.Mask))
+  )
+  (footprint "MountingHole:MountingHole_2.2mm_M2_ISO14580" (layer "F.Cu")
+    (at 123.825 47.625)
+    (descr "Mounting Hole 2.2mm, no annular, M2, ISO14580")
+    (tags "mounting hole 2.2mm no annular m2 iso14580")
+    (attr exclude_from_pos_files exclude_from_bom)
+    (fp_text reference "REF**" (at 0 -2.9) (layer "F.SilkS") hide
+      (effects (font (size 1 1) (thickness 0.15)))
+    )
+    (fp_text value "M2" (at 0 2.9) (layer "F.Fab")
+      (effects (font (size 1 1) (thickness 0.15)))
+    )
+    (fp_text user "${REFERENCE}" (at 0 0) (layer "F.Fab") hide
+      (effects (font (size 1 1) (thickness 0.15)))
+    )
+    (fp_circle (center 0 0) (end 1.9 0) (layer "Cmts.User") (width 0.15) (fill none))
+    (fp_circle (center 0 0) (end 2.15 0) (layer "F.CrtYd") (width 0.05) (fill none))
+    (pad "" np_thru_hole circle (at 0 0) (size 2.2 2.2) (drill 2.2) (layers *.Cu *.Mask))
+  )
   (footprint "Resistor_SMD:R_0402_1005Metric" (layer "F.Cu")
     (at 75.32 103.555)
@@
     )
   )
+  (footprint "MountingHole:MountingHole_2.2mm_M2_ISO14580" (layer "F.Cu")
+    (at 47.625 123.825)
+    (descr "Mounting Hole 2.2mm, no annular, M2, ISO14580")
+    (tags "mounting hole 2.2mm no annular m2 iso14580")
+    (attr exclude_from_pos_files exclude_from_bom)
+    (fp_text reference "REF**" (at 0 -2.9) (layer "F.SilkS") hide
+      (effects (font (size 1 1) (thickness 0.15)))
+    )
+    (fp_text value "M2" (at 0 2.9) (layer "F.Fab")
+      (effects (font (size 1 1) (thickness 0.15)))
+    )
+    (fp_text user "${REFERENCE}" (at 0 0) (layer "F.Fab") hide
+      (effects (font (size 1 1) (thickness 0.15)))
+    )
+    (fp_circle (center 0 0) (end 1.9 0) (layer "Cmts.User") (width 0.15) (fill none))
+    (fp_circle (center 0 0) (end 2.15 0) (layer "F.CrtYd") (width 0.05) (fill none))
+    (pad "" np_thru_hole circle (at 0 0) (size 2.2 2.2) (drill 2.2) (layers *.Cu *.Mask))
+  )
   (footprint "Octave_Library:Hot_Swap_Socket_CPG151101S11" (layer "F.Cu")
     (at 95.25 76.2)
@@
     )
   )
+  (footprint "MountingHole:MountingHole_2.2mm_M2_ISO14580" (layer "F.Cu")
+    (at 123.825 131.825)
+    (descr "Mounting Hole 2.2mm, no annular, M2, ISO14580")
+    (tags "mounting hole 2.2mm no annular m2 iso14580")
+    (attr exclude_from_pos_files exclude_from_bom)
+    (fp_text reference "REF**" (at 0 -2.9) (layer "F.SilkS") hide
+      (effects (font (size 1 1) (thickness 0.15)))
+    )
+    (fp_text value "M2" (at 0 2.9) (layer "F.Fab")
+      (effects (font (size 1 1) (thickness 0.15)))
+    )
+    (fp_text user "${REFERENCE}" (at 0 0) (layer "F.Fab") hide
+      (effects (font (size 1 1) (thickness 0.15)))
+    )
+    (fp_circle (center 0 0) (end 1.9 0) (layer "Cmts.User") (width 0.15) (fill none))
+    (fp_circle (center 0 0) (end 2.15 0) (layer "F.CrtYd") (width 0.05) (fill none))
+    (pad "" np_thru_hole circle (at 0 0) (size 2.2 2.2) (drill 2.2) (layers *.Cu *.Mask))
+  )
+  (footprint "MountingHole:MountingHole_2.2mm_M2_ISO14580" (layer "F.Cu")
+    (at 123.825 123.825)
+    (descr "Mounting Hole 2.2mm, no annular, M2, ISO14580")
+    (tags "mounting hole 2.2mm no annular m2 iso14580")
+    (attr exclude_from_pos_files exclude_from_bom)
+    (fp_text reference "REF**" (at 0 -2.9) (layer "F.SilkS") hide
+      (effects (font (size 1 1) (thickness 0.15)))
+    )
+    (fp_text value "M2" (at 0 2.9) (layer "F.Fab")
+      (effects (font (size 1 1) (thickness 0.15)))
+    )
+    (fp_text user "${REFERENCE}" (at 0 0) (layer "F.Fab") hide
+      (effects (font (size 1 1) (thickness 0.15)))
+    )
+    (fp_circle (center 0 0) (end 1.9 0) (layer "Cmts.User") (width 0.15) (fill none))
+    (fp_circle (center 0 0) (end 2.15 0) (layer "F.CrtYd") (width 0.05) (fill none))
+    (pad "" np_thru_hole circle (at 0 0) (size 2.2 2.2) (drill 2.2) (layers *.Cu *.Mask))
+  )
   (footprint "Capacitor_SMD:C_0402_1005Metric" locked (layer "F.Cu")
